Commit message: added  remaining files

File: mp_project/src/world_launch/models/coke_can.urdf (robot description, URDF)
Before this commit: robot coke_can_model, 1 links, 0 joints
Links:
- link coke_can: geometry collision mesh filename=package://world_launch/models/mesh/coke_can.dae scale=0.001 0.001 0.0025; visual mesh filename=package://world_launch/models/mesh/coke_can.dae scale=0.001 0.001 0.0025

File: mp_project/src/world_launch/models/cube_red.urdf (robot description, URDF)
Before this commit: robot simple_box, 1 links, 0 joints
Links:
- link my_box: geometry collision box size=0.058 0.058 0.3; visual box size=0.058 0.058 0.3

File: mp_project/src/world_launch/models/cylinder_green.urdf (robot description, URDF)
Before this commit: robot simple_cylinder, 1 links, 0 joints
Links:
- link my_cylinder: geometry collision cylinder length=1.089 radius=0.05; visual cylinder length=1.089 radius=0.05

File: mp_project/src/world_launch/models/table.urdf (robot description, URDF)
Before this commit: robot table, 5 links, 4 joints
Links:
- link leg2_link: geometry collision cylinder length=0.3=55 radius=0.02; visual cylinder length=0.55 radius=0.02
Joints:
- joint leg1_joint: origin xyz=0.5 1.0 0.55 rpy=0 0 0 -> xyz=0.5 1.0 0.35 rpy=0 0 0
- joint leg2_joint: origin xyz=-0.5 1.0 0.55 rpy=0 0 0 -> xyz=-0.5 1.0 0.35 rpy=0 0 0
- joint leg3_joint: origin xyz=0.5 -1.0 0.55 rpy=0 0 0 -> xyz=0.5 -1.0 0.35 rpy=0 0 0
- joint leg4_joint: origin xyz=-0.5 -1.0 0.55 rpy=0 0 0 -> xyz=-0.5 -1.0 0.35 rpy=0 0 0
